File: 24S_Counter.kicad_pcb (KiCad board)
At the start: 2 copper layers, 0 parts

Commit message: updated PCB
Parts:
- added G***: LOGO, my_footprints:geo, F.Cu at (86.0, 37.0)
- added H1: MountingHole, MountingHole:MountingHole_2.2mm_M2, F.Cu at (64.3, 35.3)
- added H2: MountingHole, MountingHole:MountingHole_2.2mm_M2, F.Cu at (139.7, 35.3)
- added H3: MountingHole, MountingHole:MountingHole_2.2mm_M2, F.Cu at (139.7, 89.7)
- added H4: MountingHole, MountingHole:MountingHole_2.2mm_M2, F.Cu at (64.3, 89.7)
- added J1: +5V, my_footprints:Terminal_Block_5mm, F.Cu at (73.5, 37.0)
- added J2: EXT_CLK, Connector_PinHeader_2.54mm:PinHeader_1x02_P2.54mm_Vertical, F.Cu at (69.5, 76.5)
- added R1: 100R, Resistor_SMD:R_1206_3216Metric_Pad1.30x1.75mm_HandSolder, F.Cu at (97.0, 49.0)
- added R10: 100R, Resistor_SMD:R_1206_3216Metric_Pad1.30x1.75mm_HandSolder, F.Cu at (130.0, 81.0)
- added R11: 100R, Resistor_SMD:R_1206_3216Metric_Pad1.30x1.75mm_HandSolder, F.Cu at (130.0, 85.0)
- added R12: 100R, Resistor_SMD:R_1206_3216Metric_Pad1.30x1.75mm_HandSolder, F.Cu at (130.0, 89.0)
- added R13: 100R, Resistor_SMD:R_1206_3216Metric_Pad1.30x1.75mm_HandSolder, F.Cu at (125.5, 42.5)
- added R14: 100R, Resistor_SMD:R_1206_3216Metric_Pad1.30x1.75mm_HandSolder, F.Cu at (119.5, 42.5)
- added R15: 1K, Resistor_SMD:R_1206_3216Metric_Pad1.30x1.75mm_HandSolder, F.Cu at (91.5, 85.5)
- added R16: 10K, Resistor_SMD:R_1206_3216Metric_Pad1.30x1.75mm_HandSolder, F.Cu at (91.5, 81.5)
- added R17: 1K, Resistor_SMD:R_1206_3216Metric_Pad1.30x1.75mm_HandSolder, F.Cu at (74.5, 80.5)
- added R18: 10K, Resistor_SMD:R_1206_3216Metric_Pad1.30x1.75mm_HandSolder, F.Cu at (74.5, 74.5)
- added R2: 100R, Resistor_SMD:R_1206_3216Metric_Pad1.30x1.75mm_HandSolder, F.Cu at (97.0, 53.0)
- added R3: 100R, Resistor_SMD:R_1206_3216Metric_Pad1.30x1.75mm_HandSolder, F.Cu at (97.0, 57.0)
- added R4: 100R, Resistor_SMD:R_1206_3216Metric_Pad1.30x1.75mm_HandSolder, F.Cu at (97.0, 61.0)
- added R5: 100R, Resistor_SMD:R_1206_3216Metric_Pad1.30x1.75mm_HandSolder, F.Cu at (97.0, 65.0)
- added R6: 100R, Resistor_SMD:R_1206_3216Metric_Pad1.30x1.75mm_HandSolder, F.Cu at (107.0, 42.5)
- added R7: 100R, Resistor_SMD:R_1206_3216Metric_Pad1.30x1.75mm_HandSolder, F.Cu at (97.0, 45.0)
- added R8: 100R, Resistor_SMD:R_1206_3216Metric_Pad1.30x1.75mm_HandSolder, F.Cu at (130.0, 73.0)
- added R9: 100R, Resistor_SMD:R_1206_3216Metric_Pad1.30x1.75mm_HandSolder, F.Cu at (130.0, 77.0)
- added SW1: EN, my_footprints:slide_switch_2.54mm, F.Cu at (81.5, 78.0)
- added SW2: RST, my_footprints:tact_switch_5mm, F.Cu at (91.5, 75.5)
- added U1: 74LS192, my_footprints:74LS192, F.Cu at (72.2, 56.0)
- added U2: 74LS192, my_footprints:74LS192, F.Cu at (104.5, 80.5)
- added U3: 74LS48, my_footprints:74LS48, F.Cu at (85.7, 56.0)
- added U4: 74LS48, my_footprints:74LS48, F.Cu at (118.3, 80.5)
- added U5: SM420561N, Display_7Segment:7SegmentLED_LTS6760_LTS6780, F.Cu at (105.8, 63.1)
- added U6: SM420561N, Display_7Segment:7SegmentLED_LTS6760_LTS6780, F.Cu at (121.4, 63.1)
Routing:
- net GND: track 0.00 -> 203.5 mm
- net /+5V: track 0.00 -> 152.6 mm, vias 0 -> 3
- net /B0: track 0.00 -> 62.3 mm
- net /Load: track 0.00 -> 61.0 mm, vias 0 -> 1
- net Net-(U4-f): track 0.00 -> 40.2 mm
- net Net-(U6-E): track 0.00 -> 40.0 mm, vias 0 -> 1
- net Net-(U1-QC): track 0.00 -> 37.9 mm
- net Net-(U2-QC): track 0.00 -> 37.3 mm
- net Net-(U4-g): track 0.00 -> 35.9 mm
- net Net-(U6-B): track 0.00 -> 32.1 mm, vias 0 -> 1
- net /CLK: track 0.00 -> 30.3 mm, vias 0 -> 1
- net Net-(U1-QA): track 0.00 -> 29.5 mm
- net Net-(U1-QD): track 0.00 -> 29.2 mm, vias 0 -> 1
- net Net-(U2-QD): track 0.00 -> 28.8 mm, vias 0 -> 1
- net Net-(U6-A): track 0.00 -> 28.2 mm, vias 0 -> 1
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Other:
- board outline added: 83 x 62 mm
- board text added: "VIGILAR"

Commit message: Update PCB
Parts:
- moved G*** 54.3 mm to (70.5, 89.0)
Other:
- board text added: "24 SECOND COUNTER"
- board text added: "COMPUTER TECHNOLOGY"
- board text added: "Design Engineer: Franz Louis Vigilar Date: 13 April 2026"
- board text added: "LUMI"
- board text removed: "VIGILAR"
